Commit message: updates no gz plugin

File: src/real_test_robot/urdf/robot_core.xacro (robot description, xacro)
@@ -42,4 +42,7 @@
     </xacro:inertial_box>
   </link>
+  <gazebo reference="chassis">
+    <material>Gazebo/Purple</material>
+  </gazebo>
   <!-- LEFT WHEEL -->
   <joint name="left_wheel_joint" type="continuous">
@@ -48,9 +51,10 @@
     <origin xyz="0 0.175 0" rpy="-${pi/2} 0 0"/>
     <axis xyz="0 0 1"/>
+    <limit effort="0.05" velocity="10.0"/>
   </joint>
   <link name="left_wheel">
     <visual>
       <geometry>
-        <cylinder radius="0.4" length="0.05" />
+        <cylinder radius="0.04" length="0.05" />
       </geometry>
       <material name="black"/>
@@ -58,5 +62,5 @@
     <collision>
       <geometry>
-        <cylinder radius="0.4" length="0.05" />
+        <sphere radius="0.5" />
       </geometry>
     </collision>
@@ -65,4 +69,7 @@
     </xacro:inertial_cylinder>
   </link>
+  <gazebo reference="left_wheel">
+    <material>Gazebo/Black</material>
+  </gazebo>
   <!-- RIGHT WHEEL -->
   <joint name="right_wheel_joint" type="continuous">
@@ -71,9 +78,10 @@
     <origin xyz="0 -0.175 0" rpy="-${pi/2} 0 0"/>
     <axis xyz="0 0 1"/>
+    <limit effort="0.05" velocity="10.0"/>
   </joint>
   <link name="right_wheel">
     <visual>
       <geometry>
-        <cylinder radius="0.4" length="0.05" />
+        <cylinder radius="0.04" length="0.05" />
       </geometry>
       <material name="black"/>
@@ -81,5 +89,5 @@
     <collision>
       <geometry>
-        <cylinder radius="0.4" length="0.05" />
+        <sphere radius="0.5" />
       </geometry>
     </collision>
@@ -88,4 +96,7 @@
     </xacro:inertial_cylinder>
   </link>
+  <gazebo reference="right_wheel">
+    <material>Gazebo/Black</material>
+  </gazebo>
   <!-- CASTER WHEEL-->
   <joint name="caster_wheel_joint" type="fixed">
@@ -110,3 +121,8 @@
     </xacro:inertial_sphere>
   </link>
+  <gazebo reference="caster_wheel">
+    <material>Gazebo/Black</material>
+    <mu1 value="0.001"/>
+    <mu2 value="0.001"/>
+  </gazebo>
 </robot>
