Commit message: adicionando SLAM, AMCL, NAV2 para concluir navegacao autonoma, tambem adicionado setup de como rodar fim a fim

File: src/real_test_robot/urdf/gazebo_control.xacro (robot description, xacro)
@@ -16,16 +16,13 @@
       <!-- OUTPUTS -->
       <frame_id>odom</frame_id>
-      <child_base_frame>base_link</child_base_frame>
+      <child_frame_id>base_link</child_frame_id>
 			<odom_topic>odom</odom_topic>
 			<tf_topic>tf</tf_topic>
-    	<publish_odom>true</publish_odom>
-      <publish_odom_tf>true</publish_odom_tf>
-    	<publish_wheel_tf>true</publish_wheel_tf>
-      </plugin>
-			<plugin name="gz::sim::systems::JointStatePublisher" filename="gz-sim-joint-state-publisher-system">
-            <topic>joint_states</topic>
-            <joint_name>left_wheel_joint</joint_name>
-            <joint_name>right_wheel_joint</joint_name>
-      </plugin>
+    </plugin>
+		<plugin name="gz::sim::systems::JointStatePublisher" filename="gz-sim-joint-state-publisher-system">
+      <topic>joint_states</topic>
+      <joint_name>left_wheel_joint</joint_name>
+      <joint_name>right_wheel_joint</joint_name>
+    </plugin>
   </gazebo>
 </robot>

File: src/real_test_robot/urdf/real_test_robot.urdf.xacro (robot description, xacro)
@@ -1,5 +1,12 @@
 <?xml version="1.0"?>
 <robot xmlns:xacro="http://www.ros.org/wiki/xacro"  name="robot">
+    <xacro:arg name="use_ros2_control" default="false"/>
     <xacro:include filename="robot_core.xacro" />
-    <xacro:include filename="gazebo_control.xacro" />
+    <xacro:include filename="lidar.xacro" />
+    <xacro:if value="$(arg use_ros2_control)">
+        <xacro:include filename="ros2_control.xacro" />
+    </xacro:if>
+    <xacro:unless value="$(arg use_ros2_control)">
+        <xacro:include filename="gazebo_control.xacro" />
+    </xacro:unless>
 </robot>

File: src/real_test_robot/urdf/robot_core.xacro (robot description, xacro)
@@ -17,4 +17,15 @@
     <color rgba="0.220 0.610 0.0244 1"/>
   </material>
+  <material name="red">
+    <color rgba="1 0 0 1"/>
+  </material>
+  <!-- BASE FOOTPRINT  -->
+  <link name="base_footprint"/>
+  <joint name="base_footprint_joint" type="fixed">
+    <parent link="base_footprint"/>
+    <child link="base_link"/>
+    <origin xyz="0 0 0" rpy="0 0 0"/>
+  </joint>
+  <!-- BASE LINK -->
   <link name="base_link"/>
   <!-- CHASSIS -->
@@ -56,5 +67,5 @@
     <visual>
       <geometry>
-        <cylinder radius="0.04" length="0.05" />
+        <cylinder radius="0.04" length="0.05"/>
       </geometry>
       <material name="black"/>
@@ -62,5 +73,5 @@
     <collision>
       <geometry>
-        <sphere radius="0.5" />
+        <sphere radius="0.04"/>
       </geometry>
     </collision>
@@ -83,5 +94,5 @@
     <visual>
       <geometry>
-        <cylinder radius="0.04" length="0.05" />
+        <cylinder radius="0.04" length="0.05"/>
       </geometry>
       <material name="black"/>
@@ -89,5 +100,5 @@
     <collision>
       <geometry>
-        <sphere radius="0.5" />
+        <sphere radius="0.04"/>
       </geometry>
     </collision>
@@ -99,5 +110,5 @@
     <material>Gazebo/Black</material>
   </gazebo>
-  <!-- CASTER WHEEL-->
+  <!-- CASTER WHEEL -->
   <joint name="caster_wheel_joint" type="fixed">
     <parent link="chassis"/>
